File: hardware/v1/DigitalStethoscope.brd (EAGLE design)
At the start: 92 x 69.5 mm, 133 parts, among them IC1 LD398533RM, IC2 LM386M-1, M1 ELECTRET_MICROPHON-F6035AP, T1 DMN3024LSD, U2 LM324PW-TSSOP14

Commit message: v1
Parts:
- R22: value 2.2k -> 4.7k
- R23: value 1.1k -> 4.7k
Changed lines of the file:
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@@
 <attribute name="PROD_ID" value="RES-07864" x="69.4" y="40.8" size="1.778" layer="27" rot="R180" display="off"/>
 </element>
-<element name="R22" library="SparkFun-Resistors" package="0603-RES" value="2.2k" x="78.9" y="46.6">
+<element name="R22" library="SparkFun-Resistors" package="0603-RES" value="4.7k" x="78.9" y="46.6">
 <attribute name="PROD_ID" value="RES-07864" x="78.9" y="46.6" size="1.778" layer="27" display="off"/>
 </element>
@@
 <attribute name="MPN" value="CC0603KRX5R6BB475" x="79.9" y="49.65" size="1.778" layer="27" rot="R180" display="off"/>
 </element>
-<element name="R23" library="SparkFun-Resistors" package="0603-RES" value="1.1k" x="69.4" y="38.1" rot="R180">
+<element name="R23" library="SparkFun-Resistors" package="0603-RES" value="4.7k" x="69.4" y="38.1" rot="R180">
 <attribute name="PROD_ID" value="RES-07864" x="69.4" y="38.1" size="1.778" layer="27" rot="R180" display="off"/>
 </element>
