File: hardware/v1/DigitalStethoscope.sch (EAGLE design)
At the start: 133 parts, among them IC1 LD398533RM, IC2 LM386M-1, M1 ELECTRET_MICROPHON-F6035AP, T1 DMN3024LSD, U2 LM324PW-TSSOP14

Commit message: v1
Parts:
- R22: value 2.2k -> 4.7k
- R23: value 1.1k -> 4.7k
Changed lines of the file:
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@@
 <part name="R19" library="SparkFun-Resistors" deviceset="390OHM1/10W1%(0603)" device="" value="100k"/>
 <part name="R20" library="SparkFun-Resistors" deviceset="390OHM1/10W1%(0603)" device="" value="100k"/>
-<part name="R22" library="SparkFun-Resistors" deviceset="390OHM1/10W1%(0603)" device="" value="2.2k"/>
+<part name="R22" library="SparkFun-Resistors" deviceset="390OHM1/10W1%(0603)" device="" value="4.7k"/>
 <part name="C30" library="Seeed-OPL-Capacitor" deviceset="CERAMIC-4.7UF-10V-10%-X5R(0603)" device="" value="1uF"/>
-<part name="R23" library="SparkFun-Resistors" deviceset="390OHM1/10W1%(0603)" device="" value="1.1k"/>
+<part name="R23" library="SparkFun-Resistors" deviceset="390OHM1/10W1%(0603)" device="" value="4.7k"/>
 <part name="C31" library="Seeed-OPL-Capacitor" deviceset="CERAMIC-4.7UF-10V-10%-X5R(0603)" device="" value="1uF"/>
 <part name="GND24" library="supply1" deviceset="GND" device=""/>
